Commit message: fix: urdf inertia, sdf cylinder tags, pose bridge, sim launch

File: src/yavuz_description/urdf/yavuz_auv.urdf.xacro (robot description, xacro)
@@ -1,113 +1,49 @@
 <?xml version="1.0"?>
-<!--
-  YAVUZ AUV - URDF/Xacro Model
-  Donanım:
-    - Gövde: Alüminyum 6061, Ø130mm x 900mm
-    - 6x DEGZ Mitras İtici (CCW, Ø90mm)
-    - 1x IMX219-170 Kamera (170° FOV)
-    - 1x Optik Kubbe (Ø100mm, polikarbonat)
-    - Jetson Nano (ana bilgisayar)
-    - Pixhawk PX4 2.4.8
-    - BMX160 IMU
-    - LiPo 22.2V 10000mAh
-  Thruster Konfigürasyonu (BlueROV2 Standard - 6DOF):
-    Horizontal (4 adet @ ±45°): surge, sway, yaw
-    Vertical (2 adet): heave, roll/pitch
-         [T0] ←45°  45°→ [T1]        (front-top view)
-           ↖           ↗
-     [Bow]==================[Stern]
-           ↙           ↘
-         [T2] ←45°  45°→ [T3]
-         [T4]         [T5]            (vertical)
--->
 <robot name="yavuz_auv" xmlns:xacro="http://www.ros.org/wiki/xacro">
-  <!-- ==================== PARAMETRELERİ ==================== -->
   <xacro:property name="body_length"  value="0.55"/>
   <xacro:property name="body_radius"  value="0.065"/>
   <xacro:property name="body_mass"    value="10.0"/>
   <xacro:property name="thruster_mass"   value="0.344"/>
-  <xacro:property name="thruster_length" value="0.113"/>
-  <xacro:property name="thruster_radius" value="0.045"/>
-  <!-- Su yoğunluğu kg/m³ -->
-  <xacro:property name="water_density" value="1000.0"/>
-  <!-- ==================== RENK TANIMLAMALARI ==================== -->
-  <material name="dark_grey">
-    <color rgba="0.2 0.2 0.2 1.0"/>
-  </material>
   <material name="blue">
     <color rgba="0.0 0.35 0.7 1.0"/>
   </material>
-  <material name="orange">
-    <color rgba="1.0 0.5 0.0 1.0"/>
+  <material name="dark_grey">
+    <color rgba="0.2 0.2 0.2 1.0"/>
   </material>
   <material name="white">
     <color rgba="0.9 0.9 0.9 1.0"/>
   </material>
-  <material name="yellow">
-    <color rgba="1.0 0.9 0.0 1.0"/>
-  </material>
-  <!-- ==================== XACRO MAKROLARı ==================== -->
-  <xacro:macro name="thruster_link" params="name">
-    <link name="${name}">
-      <inertial>
-        <mass value="${thruster_mass}"/>
-        <inertia ixx="0.001" ixy="0.0" ixz="0.0"
-                 iyy="0.001" iyz="0.0" izz="0.0005"/>
-      </inertial>
-      <visual>
-        <geometry>
-          <cylinder radius="${thruster_radius}" length="${thruster_length}"/>
-        </geometry>
-        <material name="dark_grey"/>
-      </visual>
-      <collision>
-        <geometry>
-          <cylinder radius="${thruster_radius}" length="${thruster_length}"/>
-        </geometry>
-      </collision>
-    </link>
-  </xacro:macro>
-  <xacro:macro name="thruster_joint" params="name parent x y z roll pitch yaw">
-    <joint name="${name}_joint" type="continuous">
-      <parent link="${parent}"/>
-      <child link="${name}"/>
-      <origin xyz="${x} ${y} ${z}" rpy="${roll} ${pitch} ${yaw}"/>
-      <axis xyz="0 0 1"/>
-    </joint>
-  </xacro:macro>
-  <!-- ==================== ANA GÖVDE ==================== -->
+  <!-- Dummy root link (KDL uyumluluğu için) -->
+  <link name="base_footprint"/>
+  <joint name="base_footprint_joint" type="fixed">
+    <parent link="base_footprint"/>
+    <child link="base_link"/>
+    <origin xyz="0 0 0" rpy="0 0 0"/>
+  </joint>
+  <!-- ANA GÖVDE -->
   <link name="base_link">
     <inertial>
-      <mass value="${body_mass}"/>
+      <mass value="10.0"/>
       <origin xyz="0 0 0" rpy="0 0 0"/>
       <inertia
-        ixx="0.1 " ixy="0.0" ixz="0.0"
-        iyy="0.4"  iyz="0.0"
+        ixx="0.1" ixy="0.0" ixz="0.0"
+        iyy="0.4" iyz="0.0"
         izz="0.4"/>
     </inertial>
-    <!-- Ana silindir gövde -->
     <visual>
-      <origin xyz="0 0 0" rpy="${pi/2} 0 0"/>
+      <origin xyz="0 0 0" rpy="1.5707 0 0"/>
       <geometry>
-        <cylinder radius="${body_radius}" length="${body_length}"/>
+        <cylinder radius="0.065" length="0.55"/>
       </geometry>
       <material name="blue"/>
     </visual>
     <collision>
-      <origin xyz="0 0 0" rpy="${pi/2} 0 0"/>
+      <origin xyz="0 0 0" rpy="1.5707 0 0"/>
       <geometry>
-        <cylinder radius="${body_radius}" length="${body_length}"/>
+        <cylinder radius="0.065" length="0.55"/>
       </geometry>
     </collision>
-    <!-- Optik kubbe (ön kamera) -->
-    <visual>
-      <origin xyz="0.285 0 0" rpy="0 ${pi/2} 0"/>
-      <geometry>
-        <sphere radius="0.05"/>
-      </geometry>
-      <material name="white"/>
-    </visual>
   </link>
-  <!-- ==================== IMU LINK ==================== -->
+  <!-- IMU -->
   <link name="imu_link">
     <inertial>
@@ -121,5 +57,5 @@
     <origin xyz="0 0 0" rpy="0 0 0"/>
   </joint>
-  <!-- ==================== KAMERA LINK ==================== -->
+  <!-- KAMERA -->
   <link name="camera_link">
     <inertial>
@@ -128,7 +64,5 @@
     </inertial>
     <visual>
-      <geometry>
-        <box size="0.03 0.03 0.02"/>
-      </geometry>
+      <geometry><box size="0.03 0.03 0.02"/></geometry>
       <material name="dark_grey"/>
     </visual>
@@ -139,48 +73,37 @@
     <origin xyz="0.285 0 0" rpy="0 0 0"/>
   </joint>
-  <!-- ==================== DERINLIK SENSÖR LINK ==================== -->
-  <link name="depth_sensor_link">
-    <inertial>
-      <mass value="0.01"/>
-      <inertia ixx="0.000001" ixy="0" ixz="0" iyy="0.000001" iyz="0" izz="0.000001"/>
-    </inertial>
-  </link>
-  <joint name="depth_sensor_joint" type="fixed">
-    <parent link="base_link"/>
-    <child link="depth_sensor_link"/>
-    <origin xyz="-0.1 0 -0.05" rpy="0 0 0"/>
-  </joint>
-  <!-- ==================== THRUSTER LINKLERİ ==================== -->
-  <!-- Horizontal Thruster 0: Sol-Ön -->
+  <!-- THRUSTERLAR -->
+  <xacro:macro name="thruster_link" params="name">
+    <link name="${name}">
+      <inertial>
+        <mass value="0.344"/>
+        <inertia ixx="0.001" ixy="0" ixz="0" iyy="0.001" iyz="0" izz="0.0005"/>
+      </inertial>
+      <visual>
+        <geometry><cylinder radius="0.045" length="0.113"/></geometry>
+        <material name="dark_grey"/>
+      </visual>
+    </link>
+  </xacro:macro>
+  <xacro:macro name="thruster_joint" params="name parent x y z roll pitch yaw">
+    <joint name="${name}_joint" type="fixed">
+      <parent link="${parent}"/>
+      <child link="${name}"/>
+      <origin xyz="${x} ${y} ${z}" rpy="${roll} ${pitch} ${yaw}"/>
+    </joint>
+  </xacro:macro>
   <xacro:thruster_link name="thruster0"/>
-  <xacro:thruster_joint name="thruster0" parent="base_link"
-    x="0.18" y="0.11" z="0.0"
-    roll="0" pitch="0" yaw="${pi*3/4}"/>
-  <!-- Horizontal Thruster 1: Sağ-Ön -->
+  <xacro:thruster_joint name="thruster0" parent="base_link" x="0.18" y="0.11" z="0.0" roll="0" pitch="0" yaw="2.356"/>
   <xacro:thruster_link name="thruster1"/>
-  <xacro:thruster_joint name="thruster1" parent="base_link"
-    x="0.18" y="-0.11" z="0.0"
-    roll="0" pitch="0" yaw="${-pi*3/4}"/>
-  <!-- Horizontal Thruster 2: Sol-Arka -->
+  <xacro:thruster_joint name="thruster1" parent="base_link" x="0.18" y="-0.11" z="0.0" roll="0" pitch="0" yaw="-2.356"/>
   <xacro:thruster_link name="thruster2"/>
-  <xacro:thruster_joint name="thruster2" parent="base_link"
-    x="-0.18" y="0.11" z="0.0"
-    roll="0" pitch="0" yaw="${pi/4}"/>
-  <!-- Horizontal Thruster 3: Sağ-Arka -->
+  <xacro:thruster_joint name="thruster2" parent="base_link" x="-0.18" y="0.11" z="0.0" roll="0" pitch="0" yaw="0.785"/>
   <xacro:thruster_link name="thruster3"/>
-  <xacro:thruster_joint name="thruster3" parent="base_link"
-    x="-0.18" y="-0.11" z="0.0"
-    roll="0" pitch="0" yaw="${-pi/4}"/>
-  <!-- Vertical Thruster 4: Sol -->
+  <xacro:thruster_joint name="thruster3" parent="base_link" x="-0.18" y="-0.11" z="0.0" roll="0" pitch="0" yaw="-0.785"/>
   <xacro:thruster_link name="thruster4"/>
-  <xacro:thruster_joint name="thruster4" parent="base_link"
-    x="0.12" y="0.22" z="0.0"
-    roll="0" pitch="${pi/2}" yaw="0"/>
-  <!-- Vertical Thruster 5: Sağ -->
+  <xacro:thruster_joint name="thruster4" parent="base_link" x="0.12" y="0.22" z="0.0" roll="0" pitch="1.5707" yaw="0"/>
   <xacro:thruster_link name="thruster5"/>
-  <xacro:thruster_joint name="thruster5" parent="base_link"
-    x="0.12" y="-0.22" z="0.0"
-    roll="0" pitch="${pi/2}" yaw="0"/>
-  <!-- ==================== GAZEBO SENSOR TANIMLARI ==================== -->
+  <xacro:thruster_joint name="thruster5" parent="base_link" x="0.12" y="-0.22" z="0.0" roll="0" pitch="1.5707" yaw="0"/>
+  <!-- GAZEBO SENSÖRLER -->
   <gazebo reference="imu_link">
     <sensor name="imu_sensor" type="imu">
@@ -188,5 +111,4 @@
       <update_rate>100</update_rate>
       <topic>yavuz/imu/data</topic>
-      <gz_frame_id>imu_link</gz_frame_id>
       <imu>
         <angular_velocity>
@@ -203,47 +125,3 @@
     </sensor>
   </gazebo>
-  <gazebo reference="camera_link">
-    <sensor name="front_camera" type="camera">
-      <always_on>true</always_on>
-      <update_rate>30</update_rate>
-      <topic>yavuz/camera/image_raw</topic>
-      <gz_frame_id>camera_link</gz_frame_id>
-      <camera>
-        <horizontal_fov>2.967</horizontal_fov> <!-- 170 derece -->
-        <image>
-          <width>1280</width>
-          <height>720</height>
-          <format>R8G8B8</format>
-        </image>
-        <clip>
-          <near>0.05</near>
-          <far>50</far>
-        </clip>
-      </camera>
-    </sensor>
-  </gazebo>
-  <!-- Basınç / Derinlik Sensörü (Altimetre olarak simüle edilir) -->
-  <gazebo reference="depth_sensor_link">
-    <sensor name="depth_sensor" type="altimeter">
-      <always_on>true</always_on>
-      <update_rate>50</update_rate>
-      <topic>yavuz/depth/raw</topic>
-      <gz_frame_id>depth_sensor_link</gz_frame_id>
-      <altimeter>
-        <vertical_position>
-          <noise type="gaussian"><mean>0</mean><stddev>0.005</stddev></noise>
-        </vertical_position>
-      </altimeter>
-    </sensor>
-  </gazebo>
-  <!-- Odometry (Ground Truth - simülasyon için) -->
-  <gazebo>
-    <plugin name="gz_ros2_control::GazeboSimROS2ControlPlugin"
-            filename="gz_ros2_control-system">
-      <ros>
-        <namespace>/yavuz</namespace>
-      </ros>
-      <parameters>$(find yavuz_description)/config/gz_control.yaml</parameters>
-    </plugin>
-  </gazebo>
 </robot>
